File: Project/Kestrel47.kicad_pcb (KiCad board)
At the start: 2 copper layers, 247.6 x 76.2 mm, 100 parts, among them J1 Conn_01x03, SW1 SW_Push, SW2 SW_SPDT, U1 ProMicro

Commit message: cleaned up power routing
Routing:
- net RAW: track 36.2 -> 36.9 mm, vias 4 -> 0
- net Net-(BT1-Pad2): track 33.5 -> 34.2 mm, vias 2 -> 0
- net ROW1: track 238.2 -> 238.3 mm, vias 0 -> 4

Commit message: silkscreen update
Parts:
- added G***: LOGO, LOGO, B.Cu at (203.2, 53.0)
